File: Bank65.kicad_sch (KiCad schematic)
At the start: 2 parts, among them U1 XCKU5P-FFVB676

Commit message: finishing schematic
Connections:
- no-connect marks 0 -> 7
Changed lines of the file:
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@@
 		(color 0 0 0 0)
+	)
+	(no_connect
+		(at 87.63 173.99)
+	)
+	(no_connect
+		(at 87.63 74.93)
+	)
+	(no_connect
+		(at 87.63 102.87)
+	)
+	(no_connect
+		(at 87.63 39.37)
+	)
+	(no_connect
+		(at 87.63 138.43)
+	)
+	(no_connect
+		(at 87.63 110.49)
+	)
+	(no_connect
+		(at 87.63 146.05)
 	)
 	(bus_entry
@@
 		(in_pos_files yes)
 		(dnp no)
-		(property "Reference" "#PWR0181"
+		(property "Reference" "#PWR181"
 			(at 29.21 170.18 0)
 			(hide yes)
@@
 			(project "KU5P_Core"
 				(path "/68d0ebd3-4770-4e42-a15d-94722405f64d/8a27e5b5-485e-4923-a8ca-92c1e43f1f46/460e3070-2dd4-4116-b69c-9f64446c5546/15ff1c1c-9184-4a33-bf91-4ebd928d44e3/06a63301-2179-4bc7-9324-64c7393f5dde"
-					(reference "#PWR0181")
+					(reference "#PWR181")
 					(unit 1)
 				)
@@
 		(in_pos_files yes)
 		(dnp no)
-		(property "Reference" "#PWR0111"
+		(property "Reference" "#PWR111"
 			(at 139.7 82.55 0)
 			(hide yes)
@@
 			(project "KU5P_Core"
 				(path "/68d0ebd3-4770-4e42-a15d-94722405f64d/8a27e5b5-485e-4923-a8ca-92c1e43f1f46/460e3070-2dd4-4116-b69c-9f64446c5546/15ff1c1c-9184-4a33-bf91-4ebd928d44e3/06a63301-2179-4bc7-9324-64c7393f5dde"
-					(reference "#PWR0111")
+					(reference "#PWR111")
 					(unit 1)
 				)
