File: DDR4.kicad_sch (KiCad schematic)
At the start: 13 parts, among them U2 MT40A512M16TB, U4 MT40A512M16TB

Commit message: sync works
Parts:
- added C246, C253, C254, C255, C256, C257, C270, C271, C272, C274, C275, C276: 100n, Capacitor_SMD:C_0201_0603Metric, symbol Device:C
- R33, R34: value 10k -> 1k
Connections:
- net D4_VDD: now also C246.1, C253.1, C255.1, C256.1, C270.1, C271.1, C272.1, C274.1, C275.1, C276.1
- net D4_VPP: now also C254.1, C257.1
- net GND: now also C246.2, C253.2, C254.2, C255.2, C256.2, C257.2, C270.2, C271.2, C272.2, C274.2, C275.2, C276.2
