File: Decap.kicad_sch (KiCad schematic)
At the start: 37 parts

Commit message: sync works
Parts:
- removed C161, C164: 10u, Capacitor_SMD:C_0603_1608Metric, symbol Device:C
- removed C162: 10u, Capacitor_SMD:C_0402_1005Metric, symbol Device:C
- removed C163: 47u, Capacitor_SMD:C_0603_1608Metric, symbol Device:C
- removed C165, C166, C167, C168: 100n, Capacitor_SMD:C_0201_0603Metric, symbol Device:C
