File: FAN.kicad_sch (KiCad schematic)
At the start: 5 parts, among them J4 XH 2.54, M1 Fan_4pin, Q1 DMN2040U

Commit message: finishing schematic
Parts:
- added C106: 220U, Capacitor_Tantalum_SMD:CP_EIA-7343-31_Kemet-D, symbol Device:C_Polarized
Connections:
- net +5V: now also C106.1
- net GND: now also C106.2
Changed lines of the file:
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@@
+	)
+	(junction
+		(at 162.56 64.77)
+		(diameter 0)
+		(color 0 0 0 0)
 	)
 	(junction
@@
 	)
 	(junction
+		(at 162.56 72.39)
+		(diameter 0)
+		(color 0 0 0 0)
+	)
+	(junction
 		(at 115.57 59.69)
 		(diameter 0)
@@
 	(wire
 		(pts
+			(xy 156.21 64.77) (xy 162.56 64.77)
+		)
+		(stroke
+			(width 0)
+			(type default)
+		)
+	)
+	(wire
+		(pts
 			(xy 115.57 59.69) (xy 115.57 60.96)
 		)
@@
 	(wire
 		(pts
+			(xy 162.56 73.66) (xy 162.56 72.39)
+		)
+		(stroke
+			(width 0)
+			(type default)
+		)
+	)
+	(wire
+		(pts
 			(xy 106.68 99.06) (xy 106.68 100.33)
 		)
@@
 	(wire
 		(pts
+			(xy 156.21 72.39) (xy 162.56 72.39)
+		)
+		(stroke
+			(width 0)
+			(type default)
+		)
+	)
+	(wire
+		(pts
 			(xy 118.11 88.9) (xy 114.3 88.9)
 		)
@@
 	(wire
 		(pts
-			(xy 162.56 60.96) (xy 162.56 67.31)
+			(xy 162.56 60.96) (xy 162.56 64.77)
 		)
 		(stroke
@@
 		(pts
 			(xy 106.68 93.98) (xy 106.68 99.06)
+		)
+		(stroke
+			(width 0)
+			(type default)
+		)
+	)
+	(wire
+		(pts
+			(xy 162.56 64.77) (xy 162.56 67.31)
 		)
 		(stroke
@@
 		(in_pos_files yes)
 		(dnp no)
-		(property "Reference" "#PWR0155"
+		(property "Reference" "#PWR155"
 			(at 115.57 59.69 0)
 			(hide yes)
@@
 			(project "KU5P_Core"
 				(path "/68d0ebd3-4770-4e42-a15d-94722405f64d/8a27e5b5-485e-4923-a8ca-92c1e43f1f46/4b7b0b80-c290-42cb-8173-d9a2e211585a/91a58e44-8dd7-4a61-82ce-416c04582528"
-					(reference "#PWR0155")
+					(reference "#PWR155")
 					(unit 1)
 				)
@@
 		(dnp no)
 		(fields_autoplaced yes)
-		(property "Reference" "#PWR0156"
+		(property "Reference" "#PWR156"
 			(at 115.57 82.55 0)
 			(hide yes)
@@
 			(project "KU5P_Core"
 				(path "/68d0ebd3-4770-4e42-a15d-94722405f64d/8a27e5b5-485e-4923-a8ca-92c1e43f1f46/4b7b0b80-c290-42cb-8173-d9a2e211585a/91a58e44-8dd7-4a61-82ce-416c04582528"
-					(reference "#PWR0156")
+					(reference "#PWR156")
 					(unit 1)
 				)
@@
 	(symbol
 		(lib_id "dfdtc_power:GND")
-		(at 162.56 72.39 0)
+		(at 162.56 73.66 0)
 		(mirror y)
 		(unit 1)
@@
 		(in_pos_files yes)
 		(dnp no)
-		(property "Reference" "#PWR0204"
-			(at 162.56 78.74 0)
+		(property "Reference" "#PWR204"
+			(at 162.56 80.01 0)
 			(hide yes)
 			(show_name no)
@@
 		)
 		(property "Value" "GND"
-			(at 162.56 76.2 0)
+			(at 162.56 77.47 0)
 			(show_name no)
 			(do_not_autoplace no)
@@
 		)
 		(property "Footprint" ""
-			(at 162.56 72.39 0)
+			(at 162.56 73.66 0)
 			(hide yes)
 			(show_name no)
@@
 		)
 		(property "Datasheet" ""
-			(at 162.56 72.39 0)
+			(at 162.56 73.66 0)
 			(hide yes)
 			(show_name no)
@@
 		)
 		(property "Description" "Power symbol creates a global label with name \"GND\" , ground"
-			(at 162.56 72.39 0)
+			(at 162.56 73.66 0)
 			(hide yes)
 			(show_name no)
@@
 			(project "KU5P_Core"
 				(path "/68d0ebd3-4770-4e42-a15d-94722405f64d/8a27e5b5-485e-4923-a8ca-92c1e43f1f46/4b7b0b80-c290-42cb-8173-d9a2e211585a/91a58e44-8dd7-4a61-82ce-416c04582528"
-					(reference "#PWR0204")
+					(reference "#PWR204")
+					(unit 1)
+				)
+			)
+		)
+	)
+	(symbol
+		(lib_id "Device:C_Polarized")
+		(at 156.21 68.58 0)
+		(unit 1)
+		(body_style 1)
+		(exclude_from_sim no)
+		(in_bom yes)
+		(on_board yes)
+		(in_pos_files yes)
+		(dnp no)
+		(property "Reference" "C106"
+			(at 156.464 66.294 0)
+			(show_name no)
+			(do_not_autoplace no)
+			(effects
+				(font
+					(size 1.27 1.27)
+				)
+				(justify left)
+			)
+		)
+		(property "Value" "220U"
+			(at 156.464 71.12 0)
+			(show_name no)
+			(do_not_autoplace no)
+			(effects
+				(font
+					(size 1.27 1.27)
+				)
+				(justify left)
+			)
+		)
+		(property "Footprint" "Capacitor_Tantalum_SMD:CP_EIA-7343-31_Kemet-D"
+			(at 157.1752 72.39 0)
+			(hide yes)
+			(show_name no)
+			(do_not_autoplace no)
+			(effects
+				(font
+					(size 1.27 1.27)
+				)
+			)
+		)
+		(property "Datasheet" ""
+			(at 156.21 68.58 0)
+			(hide yes)
+			(show_name no)
+			(do_not_autoplace no)
+			(effects
+				(font
+					(size 1.27 1.27)
+				)
+			)
+		)
+		(property "Description" "Polarized capacitor"
+			(at 156.21 68.58 0)
+			(hide yes)
+			(show_name no)
+			(do_not_autoplace no)
+			(effects
+				(font
+					(size 1.27 1.27)
+				)
+			)
+		)
+		(pin "2"
+		)
+		(pin "1"
+		)
+		(instances
+			(project "KU5P_Core"
+				(path "/68d0ebd3-4770-4e42-a15d-94722405f64d/8a27e5b5-485e-4923-a8ca-92c1e43f1f46/4b7b0b80-c290-42cb-8173-d9a2e211585a/91a58e44-8dd7-4a61-82ce-416c04582528"
+					(reference "C106")
 					(unit 1)
 				)
@@
 		(in_pos_files yes)
 		(dnp no)
-		(property "Reference" "#PWR0203"
+		(property "Reference" "#PWR203"
 			(at 162.56 64.77 0)
 			(hide yes)
@@
 			(project "KU5P_Core"
 				(path "/68d0ebd3-4770-4e42-a15d-94722405f64d/8a27e5b5-485e-4923-a8ca-92c1e43f1f46/4b7b0b80-c290-42cb-8173-d9a2e211585a/91a58e44-8dd7-4a61-82ce-416c04582528"
-					(reference "#PWR0203")
+					(reference "#PWR203")
 					(unit 1)
 				)
@@
 		(in_pos_files yes)
 		(dnp no)
-		(property "Reference" "#PWR0158"
+		(property "Reference" "#PWR158"
 			(at 106.68 106.68 0)
 			(hide yes)
@@
 			(project "KU5P_Core"
 				(path "/68d0ebd3-4770-4e42-a15d-94722405f64d/8a27e5b5-485e-4923-a8ca-92c1e43f1f46/4b7b0b80-c290-42cb-8173-d9a2e211585a/91a58e44-8dd7-4a61-82ce-416c04582528"
-					(reference "#PWR0158")
+					(reference "#PWR158")
 					(unit 1)
 				)

Commit message: sync works
Parts:
- C106, J4: now not fitted; now left out of the parts list
Changed lines of the file:
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@@
 		(unit 1)
 		(body_style 1)
-		(exclude_from_sim no)
-		(in_bom yes)
-		(on_board yes)
-		(in_pos_files yes)
-		(dnp no)
+		(exclude_from_sim yes)
+		(in_bom no)
+		(on_board no)
+		(in_pos_files no)
+		(dnp yes)
 		(fields_autoplaced yes)
 		(property "Reference" "J4"
@@
 		(unit 1)
 		(body_style 1)
-		(exclude_from_sim no)
-		(in_bom yes)
-		(on_board yes)
-		(in_pos_files yes)
-		(dnp no)
+		(exclude_from_sim yes)
+		(in_bom no)
+		(on_board no)
+		(in_pos_files no)
+		(dnp yes)
 		(property "Reference" "C106"
 			(at 156.464 66.294 0)
