File: FPGA_Power.kicad_sch (KiCad schematic)
At the start: 20 parts, among them U1 XCKU5P-FFVB676

Commit message: sync works
Parts:
- removed C235, C236, C237, C238: 100n, Capacitor_SMD:C_0201_0603Metric, symbol Device:C
- removed FB2: 600@100MHz, Inductor_SMD:L_0603_1608Metric, symbol Device:FerriteBead_Small
- removed NT3: NetTie_2, NetTie:NetTie-2_SMD_Pad0.5mm, symbol Device:NetTie_2
- removed R23, R26, R28, R30: 1k, Capacitor_SMD:C_0201_0603Metric, symbol Device:R
Connections:
- net +1V2: now also R46.1, U1.AD8 (MGTAVTTRCAL_R)
- net GND: now also U1.N13 (GNDADC)
