File: FPGA_SYS.kicad_sch (KiCad schematic)
At the start: 23 parts, among them J1 GH1.25 6P, J2 GH1.25_2P, M1 Fan_4pin, Q1 DMN2040U, SW1 SW_DIP_x03, SW2 6x3.6, U1 XCKU5P-FFVB676, U5 TXB0106RGY, U6 GD25LB256

Commit message: <feat>: Modified Power Tree
Parts:
- removed C73: 220U, Capacitor_Tantalum_SMD:CP_EIA-7343-31_Kemet-D, symbol Device:C_Polarized
- removed M1: Fan_4pin, Connector:FanPinHeader_1x04_P2.54mm_Vertical, symbol Motor:Fan_4pin
- removed Q1: DMN2040U, Package_TO_SOT_SMD:SOT-23, symbol Transistor_FET:DMN2041L
- removed R45: 10K, Resistor_SMD:R_0201_0603Metric, symbol Device:R
Connections:
- no-connect marks 2 -> 1
Other:
- added sheet FAN (FAN.kicad_sch)

Commit message: sync works
Parts:
- removed C233: 100n, Capacitor_SMD:C_0201_0603Metric, symbol Device:C
- removed J2: GH1.25_2P, symbol Connector_Generic_MountingPin:Conn_01x02_MountingPin
- removed SW1: SW_DIP_x03, Button_Switch_SMD:SW_DIP_SPSTx03_Slide_6.7x9.18mm_W6.73mm_P2.54mm_LowProfile_JPin, symbol Switch:SW_DIP_x03
- removed SW2: 6x3.6, Button_Switch_SMD:SW_SPST_CK_RS282G05A3, symbol Switch:SW_Push
- added R64, R65, R66: 0, Resistor_SMD:R_0402_1005Metric, symbol Device:R
- added R67: 4.7K, Resistor_SMD:R_0201_0603Metric, symbol Device:R
- J1: footprint Connector_JST:JST_GH_BM06B-GHS-TBT_1x06-1MP_P1.25mm_Vertical -> Connector_JST:JST_GH_SM06B-GHS-TB_1x06-1MP_P1.25mm_Horizontal
- R36: footprint Resistor_SMD:R_0603_1608Metric -> Resistor_SMD:R_0402_1005Metric
- RN8: value 10k -> 1k
Connections:
- net VCCO_HP is gone; now on net VCCO_0: RN8.5 (R4.2), RN8.6 (R3.2), RN8.7 (R2.2), RN8.8 (R1.2)
- net DONE_0: now also U5.6 (A5); no longer U5.7 (A6)
- net GND: now also U1.T13 (DXN), U1.T14 (DXP), R64.1, R65.1, R66.1
- net SYS_PG: now also U5.10 (B6); no longer U5.11 (B5)
- net SYS_PG_IO: now also U5.7 (A6); no longer U5.6 (A5)
- net TDO_IO: now also U5.3 (A2); no longer U5.5 (A4)
- net TMS_IO: now also U5.5 (A4); no longer U5.3 (A2)
- net VCCO_0: now also R67.2
- net at R44.1: now also U5.11 (B5); no longer U5.10 (B6)
- net TDO_0_SV: now reaches D1.4 (K), J1.3 (Pin_3)
- net TDO_0_SV: now also U5.14 (B2); no longer U5.13 (B3)
- net TCK_0_SV: now reaches D1.5 (K), J1.4 (Pin_4)
- net TCK_0_SV: now also U5.16 (B1); no longer U5.12 (B4)
- net PROGRAM_B_0: now reaches U1.AB9 (PROGRAM_B_0)
- net PROGRAM_B_0: now also R67.1
- net at RN8.4 (R4.1), U1.AF12 (M2_0): now also R66.2
- net at RN8.3 (R3.1), U1.AA9 (M1_0): now also R65.2
- net at RN8.2 (R2.1), U1.AA10 (M0_0): now also R64.2
- new net TDI_0_SV: D1.1 (K), J1.2 (Pin_2), U5.13 (B3)
- new net TMS_0_SV: D1.3 (K), J1.1 (Pin_1), U5.12 (B4)
Other:
- moved on the sheet: C169, C173, D1, D2, J1, R36, R44, RN8, U6
