File: KU5P_Core.kicad_sch (KiCad schematic)
At the start: 0 parts

Commit message: finishing schematic
Other:
- removed sheet B2B_CONN
Changed lines of the file:
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@@
 	(paper "A4")
-	(sheet
-		(at 36.83 39.37)
-		(size 12.7 39.37)
-		(exclude_from_sim no)
-		(in_bom yes)
-		(on_board yes)
-		(dnp no)
-		(fields_autoplaced yes)
-		(stroke
-			(width 0.1524)
-			(type solid)
-		)
-		(fill
-			(color 0 0 0 0)
-		)
-		(property "Sheetname" "B2B_CONN"
-			(at 36.83 38.6584 0)
-			(show_name no)
-			(do_not_autoplace no)
-			(effects
-				(font
-					(size 1.27 1.27)
-				)
-				(justify left bottom)
-			)
-		)
-		(property "Sheetfile" "B2B_CONN.kicad_sch"
-			(at 36.83 79.3246 0)
-			(show_name no)
-			(do_not_autoplace no)
-			(effects
-				(font
-					(size 1.27 1.27)
-				)
-				(justify left top)
-			)
-		)
-		(instances
-			(project "KU5P_Core"
-				(path "/68d0ebd3-4770-4e42-a15d-94722405f64d"
-					(page "23")
-				)
-			)
-		)
-	)
 	(sheet
 		(at 73.66 63.5)

Commit message: sync works
Parts:
- added H1, H2, H3, H4: M3, MountingHole:MountingHole_3mm_Pad_TopBottom, symbol Mechanical:MountingHole_Pad
Connections:
- new net GND: H1.1, H2.1, H3.1, H4.1
