File: P1.kicad_sch (KiCad schematic)
At the start: 50 parts, among them IC3 PMIC_P1

Commit message: <feat>: Modified Power Tree
Parts:
- added C105: 4.7u, Resistor_SMD:R_0603_1608Metric, symbol Device:C
- added C246: 100n, Capacitor_SMD:C_0603_1608Metric, symbol Device:C
- added U7: SiP32508DT, Package_TO_SOT_SMD:TSOT-23-6, symbol Power_Management:SiP32508DT
- C97: now not fitted; now left out of the parts list
Connections:
- net 1V8: now also C105.1, U7.5 (IN), U7.6 (IN); no longer IC3.12 (SWIN)
- net 3V3: now also IC3.12 (SWIN), IC3.17 (DLDOIN1), IC3.29 (DLDOIN2)
- net GND: now also C105.2, C246.2, U7.4 (GND)
- net GPIO: now also IC3.49 (GPIO3); no longer IC3.51 (GPIO2)
- net VCCO_0: now also C246.1, U7.1 (OUT), U7.2 (OUT); no longer C97.1, IC3.30 (DLDO7)
- net VCCO_HD: no longer C195.1, C198.1, L13.1, NT11.1
- net VSYS: no longer IC3.17 (DLDOIN1), IC3.29 (DLDOIN2)
- net MGTVCCAUX renamed VCCO_HD87
- new net: C97.1, IC3.30 (DLDO7)
- new net VCCO0_EN: IC3.51 (GPIO2), U7.3 (EN)
- new net VCCO_HP: C195.1, C198.1, L13.1, NT11.1
- no-connect marks 17 -> 16

Commit message: modified Power config
Parts:
- added C247, C248, C249, C250, C251, C252: 22u, Capacitor_SMD:C_0805_2012Metric, symbol Device:C
- L13, L14, L15, L16, L17, L18: footprint Inductor_SMD:L_Changjiang_FXL0420 -> Inductor_SMD:L_Changjiang_FTC252012S
Connections:
- net 0V9: now also C247.1
- net 1V2: now also C252.1
- net 1V8: now also C249.1
- net 3V3: now also C250.1
- net GND: now also C247.2, C248.2, C249.2, C250.2, C251.2, C252.2
- net VCCO_HD: now also C251.1
- net VCCO_HP: now also C248.1

Commit message: finishing schematic
Connections:
- net PMIC_32KOUT: now reaches IC3.50 (32KOUT)
- no-connect marks 16 -> 15
Changed lines of the file:
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@@
 	)
 	(no_connect
-		(at 195.58 91.44)
-	)
-	(no_connect
 		(at 71.12 152.4)
 	)
@@
 		)
 	)
+	(global_label "PMIC_32KOUT"
+		(shape output)
+		(at 195.58 91.44 180)
+		(effects
+			(font
+				(size 1.27 1.27)
+			)
+			(justify right)
+		)
+		(property "Intersheetrefs" "${INTERSHEET_REFS}"
+			(at 195.58 91.44 0)
+			(hide yes)
+			(show_name no)
+			(do_not_autoplace no)
+			(effects
+				(font
+					(size 1.27 1.27)
+				)
+			)
+		)
+	)
 	(hierarchical_label "VCCO_HD87"
 		(shape output)
@@
 		(dnp no)
 		(fields_autoplaced yes)
-		(property "Reference" "#PWR047"
+		(property "Reference" "#PWR47"
 			(at 180.34 157.48 0)
 			(hide yes)
@@
 			(project "KU5P_Core"
 				(path "/68d0ebd3-4770-4e42-a15d-94722405f64d/ca568b1d-a558-4336-b7e2-be12f8fb35d1/6988b94f-4fe9-4a8a-87b3-ac7dbeb7ca47"
-					(reference "#PWR047")
+					(reference "#PWR47")
 					(unit 1)
 				)

Commit message: sync works
Parts:
- removed C218, C246: 100n, Capacitor_SMD:C_0603_1608Metric, symbol Device:C
- removed C221: 100u, Capacitor_Tantalum_SMD:CP_EIA-7343-20_Kemet-V, symbol Device:C_Polarized
- removed C97: 10u, Resistor_SMD:R_0603_1608Metric, symbol Device:C
- removed NT10, NT11, NT4, NT5, NT6, NT7, NT8, NT9: NetTie_2, NetTie:NetTie-2_SMD_Pad0.5mm, symbol Device:NetTie_2
- removed U7: SiP32508DT, Package_TO_SOT_SMD:TSOT-23-6, symbol Power_Management:SiP32508DT
- added C107, C62: 10u, Capacitor_SMD:C_0402_1005Metric, symbol Device:C
- added C262, C263, C264, C265, C266, C267: 22u, Capacitor_SMD:C_0402_1005Metric, symbol Device:C
- C105: value 4.7u -> 10u; footprint Resistor_SMD:R_0603_1608Metric -> Capacitor_SMD:C_0402_1005Metric
- C194, C195, C196, C197, C198, C199, C206, C207, C208, C210, C211, C212, C247, C248, C249, C250, C251, C252: footprint Capacitor_SMD:C_0805_2012Metric -> Capacitor_SMD:C_0402_1005Metric
- C200, C202, C204, C209, C214, C216: value 100n -> 22u; footprint Capacitor_SMD:C_0603_1608Metric -> Capacitor_SMD:C_0402_1005Metric
- C201, C203, C205, C213, C215, C217, C220: footprint Capacitor_SMD:C_0805_2012Metric -> Capacitor_SMD:C_0603_1608Metric
- C219: footprint Capacitor_SMD:C_0603_1608Metric -> Capacitor_SMD:C_0402_1005Metric
- C92, C95, C98: footprint Resistor_SMD:R_0603_1608Metric -> Capacitor_SMD:C_0402_1005Metric
Connections:
- net 0V9: now also C202.1, IC3.11 (FB4), C263.1
- net 1V2: now also C216.1, IC3.39 (FB1), C267.1
- net 1V8: now also C207.1, C211.1, C214.1, C250.1, IC3.34 (FB2), L17.1, C266.1; no longer C105.1, C196.1, C199.1, C249.1, L15.1
- net 3V3: now also C105.1, C107.1; no longer C207.1, C211.1, C250.1, L17.1
- net GND: now also IC3.40 (FB1GND), IC3.5 (FB3GND), C107.2, C262.2, C263.2, C264.2, C265.2, C266.2, C267.2, C62.2
- net VCCO_0: now also C196.1, C199.1, C200.1, C249.1, IC3.6 (FB3), L15.1, C262.1
- net VCCO_HD: now also C209.1, IC3.25 (FB5), C265.1
- net VCCO_HP: now also C204.1, IC3.20 (FB6), C264.1
- net VSYS: no longer C200.1, C202.1, C204.1, C209.1, C214.1, C216.1
- net MGTVCCAUX: now reaches IC3.30 (DLDO7)
- net MGTVCCAUX: now also C62.1
Other:
- moved on the sheet: C98
