File: Power.kicad_sch (KiCad schematic)
At the start: 6 parts, among them SW3 6x3.6, U3 LP5912-1.5DRV

Commit message: <feat>: Modified Power Tree
Other:
- sheet 5V_Rail ports: added 3V3O, Vin; removed 12Vin
- sheet P1 ports: added VCCO_HD87; removed none
Changed lines of the file:
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@@
 	(wire
 		(pts
+			(xy 123.19 158.75) (xy 237.49 158.75)
+		)
+		(stroke
+			(width 0)
+			(type default)
+		)
+	)
+	(wire
+		(pts
 			(xy 105.41 125.73) (xy 105.41 128.27)
 		)
@@
 		)
 	)
+	(label "VCCO_87"
+		(at 149.86 158.75 180)
+		(effects
+			(font
+				(size 1.27 1.27)
+			)
+			(justify right bottom)
+		)
+	)
 	(label "0V85"
 		(at 149.86 110.49 180)
@@
 	)
 	(symbol
+		(lib_id "dfdtc_power:+1V8")
+		(at 237.49 158.75 0)
+		(unit 1)
+		(body_style 1)
+		(exclude_from_sim no)
+		(in_bom yes)
+		(on_board yes)
+		(in_pos_files yes)
+		(dnp no)
+		(fields_autoplaced yes)
+		(property "Reference" "#PWR0194"
+			(at 237.49 162.56 0)
+			(hide yes)
+			(show_name no)
+			(do_not_autoplace no)
+			(effects
+				(font
+					(size 1.27 1.27)
+				)
+			)
+		)
+		(property "Value" "VCCO_HD87"
+			(at 237.49 153.67 0)
+			(show_name no)
+			(do_not_autoplace no)
+			(effects
+				(font
+					(size 1.27 1.27)
+				)
+			)
+		)
+		(property "Footprint" ""
+			(at 237.49 158.75 0)
+			(hide yes)
+			(show_name no)
+			(do_not_autoplace no)
+			(effects
+				(font
+					(size 1.27 1.27)
+				)
+			)
+		)
+		(property "Datasheet" ""
+			(at 237.49 158.75 0)
+			(hide yes)
+			(show_name no)
+			(do_not_autoplace no)
+			(effects
+				(font
+					(size 1.27 1.27)
+				)
+			)
+		)
+		(property "Description" "Power symbol creates a global label with name \"+1V8\""
+			(at 237.49 158.75 0)
+			(hide yes)
+			(show_name no)
+			(do_not_autoplace no)
+			(effects
+				(font
+					(size 1.27 1.27)
+				)
+			)
+		)
+		(pin "1"
+		)
+		(instances
+			(project "KU5P_Core"
+				(path "/68d0ebd3-4770-4e42-a15d-94722405f64d/ca568b1d-a558-4336-b7e2-be12f8fb35d1"
+					(reference "#PWR0194")
+					(unit 1)
+				)
+			)
+		)
+	)
+	(symbol
 		(lib_id "dfdtc_power:+1V2")
 		(at 171.45 140.97 0)
@@
 			)
 		)
+		(pin "VCCO_HD87" output
+			(at 123.19 158.75 0)
+			(effects
+				(font
+					(size 1.27 1.27)
+				)
+				(justify right)
+			)
+		)
 		(instances
 			(project "KU5P_Core"
@@
 	(sheet
 		(at 55.88 134.62)
-		(size 17.78 7.62)
+		(size 17.78 15.24)
 		(exclude_from_sim yes)
 		(in_bom no)
@@
 		)
 		(property "Sheetfile" "5V_Rail.kicad_sch"
-			(at 55.88 142.8246 0)
+			(at 55.88 150.4446 0)
 			(hide yes)
 			(show_name no)
@@
 			)
 		)
-		(pin "12Vin" input
+		(pin "3V3O" output
+			(at 73.66 142.24 0)
+			(effects
+				(font
+					(size 1.27 1.27)
+				)
+				(justify right)
+			)
+		)
+		(pin "Vin" input
 			(at 55.88 137.16 180)
 			(effects

Commit message: finishing schematic
Connections:
- net P1/PWRKY renamed PMIC_PWRKY

Commit message: sync works
Parts:
- removed C234: 100n, Capacitor_SMD:C_0603_1608Metric, symbol Device:C
- removed SW3: 6x3.6, Button_Switch_SMD:SW_SPST_CK_RS282G05A3, symbol Switch:SW_Push
Other:
- sheet 5V_Rail renamed IN_Rail
- sheet IN_Rail ports: added none; removed 5VO
