File: VCCINT.kicad_sch (KiCad schematic)
At the start: 88 parts

Commit message: sync works
Parts:
- removed C62, C64, C66: 100u, Capacitor_Tantalum_SMD:CP_EIA-7343-20_Kemet-V, symbol Device:C_Polarized
- added NT12, NT13, NT14: NetTie_2, NetTie:NetTie-2_SMD_Pad0.5mm, symbol Device:NetTie_2
- C19, C20, C21, C23, C27, C28, C36, C37, C45, C47, C55, C56, C58, C61: footprint Capacitor_SMD:C_1206_3216Metric -> Capacitor_SMD:C_0603_1608Metric
- C22, C24, C25, C26, C29, C30, C31, C32, C33, C34, C35, C38, C39, C40, C41, C42, C43, C44, C46, C48, C49, C50, C51, C52, C53, C54, C57, C59, C63, C65: footprint Capacitor_SMD:C_1206_3216Metric -> Capacitor_SMD:C_0805_2012Metric
- C60: value 100u -> 470u
- NT1, NT2: footprint (none) -> NetTie:NetTie-2_SMD_Pad0.5mm
Connections:
- net GND: now also NT12.2, NT13.2, NT14.2
- net GNDA: now also NT12.1, NT13.1, NT14.1
- net VCC_M: no longer C72.1, IC2.17 (VCC), R4.1
- new net VCC_S: C72.1, IC2.17 (VCC), R4.1
